Commit message: add torque_controller

File: xacro/mmm_robot.xacro (robot description, xacro)
@@ -7,4 +7,9 @@
     <color rgba="1.0 0.0 0.0 2.5"/>
   </material>
+  <gazebo>
+    <plugin name="gazebo_ros_control" filename="libgazebo_ros_control.so">
+      <robotNamespace>/mmm_robot</robotNamespace>
+    </plugin>
+  </gazebo>
   <xacro:macro name="wheel_macro" params="parent prefix xyz">
     <joint name="${prefix}_joint" type="continuous">
@@ -16,11 +21,11 @@
     <transmission name="${prefix}_trans" type="SimpleTransmission">
       <type>transmission_interface/SimpleTransmission</type>
+        <joint name="${prefix}_joint">
+          <hardwareInterface>hardware_interface/EffortJointInterface</hardwareInterface>
+        </joint>
         <actuator name="${prefix}_motor">
           <hardwareInterface>hardware_interface/EffortJointInterface</hardwareInterface>
           <mechanicalReduction>1</mechanicalReduction>
         </actuator>
-      <joint name="${prefix}_joint">
-        <hardwareInterface>hardware_interface/EffortJointInterface</hardwareInterface>
-      </joint>
     </transmission>
     <link name="${prefix}_link">
@@ -107,8 +112,3 @@
     <mu2 value="0.5" />
   </gazebo>
-  <gazebo>
-    <plugin name="gazebo_ros_control" filename="libgazebo_ros_control.so">
-      <robotNamespace>/mmm_robot</robotNamespace>
-    </plugin>
-  </gazebo>
 </robot>
